File: voltage_and_current_measurement.kicad_sch (KiCad schematic)
At the start: 71 parts, among them IC1 VIA2000SD, J4 V_bat_in, J5 V_bat_out, U16 CZ3A05, U2 ACS37030LLZATR-065B3, U3 OPA2328DR, U4 OPA2328DR

Commit message: Commit before 5V rebase.
[KiCad Version: 10.0.4]
Parts:
- added ACSVref1, CurSig1: TestPoint, TestPoint:TestPoint_Pad_D1.0mm, symbol Connector:TestPoint
- added C10, C7, C8, C9: 1000u, Capacitor_THT:C_Radial_D8.0mm_H11.5mm_P3.50mm, symbol Device:C
- added C4, C5, C6: 1u, Capacitor_SMD:C_0603_1608Metric_Pad1.08x0.95mm_HandSolder, symbol Device:C
- added D1, D2: 1.5SMCxxCA, Diode_SMD:D_SMC, symbol Diode:1.5SMCxxCA
- added J5: V_bat_in, custom_footprints:AMASS_XT60PW-M_1x02_P7.20mm_Horizontal_with3DModel, symbol Connector:Conn_01x02_Pin
- added J6: V_bat_out, custom_footprints:AMASS_XT60PW-M_1x02_P7.20mm_Horizontal_with3DModel, symbol Connector:Conn_01x02_Pin
- renumbered ACSVref1 to ACSVref2, C12 to C11, C4 to C12, C5 to C13, C6 to C14, C7 to C15, C17 to C16, C8 to C17, C9 to C18, C10 to C19, C11 to C20, C13 to C21, C14 to C22, C15 to C23, C16 to C24, C18 to C25, C19 to C26, C20 to C27, C21 to C28, C22 to C29, C23 to C30, C24 to C31, C25 to C32, C26 to C33, C27 to C34, C28 to C35, C29 to C36, C30 to C37, C31 to C38, C32 to C39, C33 to C40, CurSig1 to CurSig2, D1 to D3, D2 to D4, J4 to J7, J5 to J8, R11 to R10, R12 to R11, R13 to R12, R14 to R13, R15 to R14, R16 to R15, R17 to R16, R18 to R17, R19 to R18, R20 to R19, R5 to R4, R6 to R5, R7 to R6, R8 to R7, R9 to R8, R10 to R9, U16 to U3, U3 to U4, U4 to U5
Connections:
- net +3V3_Ana: now also C4.1, C5.1, C6.1
- net ACS_VREF: now also ACSVref1.1
- net GND: now also C4.2, C5.2, C6.2
- net GND_ISO: now also C10.2, C7.2, C8.2, C9.2, D1.1 (A1), D2.1 (A1), J5.1 (Pin_1), J6.1 (Pin_1)
- net V_bat_in: now also U3.1 (IP), C10.1, C8.1, D1.2 (A2), J5.2 (Pin_2)
- net V_bat_out: now also U3.5 (IN), C7.1, C9.1, D2.2 (A2), J6.2 (Pin_2)
- net cur_sig: now also CurSig1.1
Other:
- moved on the sheet: ACSVref2, C15, C17, C18, CurSig2, D3, D4, J7, J8, U3

Commit message: Implemented SAR ADC Buffering on top layer with one OPA387
[KiCad Version: 10.0.4]
Parts:
- removed R12, R13: 3.32k, Resistor_SMD:R_0603_1608Metric_Pad0.98x0.95mm_HandSolder, symbol Device:R
- removed R8, R9: 2.37k, Resistor_SMD:R_0603_1608Metric_Pad0.98x0.95mm_HandSolder, symbol Device:R
- added C35, C42: 1u, Capacitor_SMD:C_0603_1608Metric_Pad1.08x0.95mm_HandSolder, symbol Device:C
- added R10, R11: 2.37k, Resistor_SMD:R_0603_1608Metric_Pad0.98x0.95mm_HandSolder, symbol Device:R
- added R14: 3.32k, Resistor_SMD:R_0603_1608Metric_Pad0.98x0.95mm_HandSolder, symbol Device:R
- added R18: 22R, Resistor_SMD:R_0603_1608Metric_Pad0.98x0.95mm_HandSolder, symbol Device:R
- ACSVref1, C2, C3, C4, C5, C6, CurSig1, D1, D2, J5, J6, U2: now left out of the parts list
- R15: value 22R -> 3.32k
- renumbered C12 to C11, C13 to C12, C14 to C13, C15 to C14, C17 to C15, C18 to C16, C19 to C17, C20 to C18, C21 to C19, C22 to C20, C23 to C21, C24 to C22, C25 to C23, C26 to C24, C27 to C25, C28 to C26, C29 to C27, C30 to C28, C31 to C29, C32 to C30, C33 to C31, C34 to C32, C35 to C33, C36 to C34, C11 to C36, C16 to C41, IC1 to IC2, R10 to R12, R11 to R13, R14 to R16, R16 to R19, R18 to R20, R19 to R21, R4 to R6, R5 to R7, R6 to R8, R7 to R9
Connections:
- net +3V3_Ana: no longer C14.1, C15.1, C16.1, C17.1, C18.1, C36.1, C41.1, IC2.8 (VDD2), U3.13 (VDD), U4.8 (V+), U5.8 (V+)
- net ACS_VREF: now also U3.11 (OCD2)
- net GND: now also C35.2, C42.2
- net V_sig: now also R10.1
- net Vout_ref: now also R11.1
- net cur_sig: now also U3.12 (VOUT)
- net at C25.1: now also R10.2, R14.1
- net at C21.1, U5.3 (+): now also R14.2
- net at C30.1, MCP2.4 (AIN-): now also R18.2; no longer R15.2
- net at C26.2, U5.6 (-), U5.7: now also R18.1; no longer R15.1
- net at C26.1: now also R15.1, R11.2
- net at C22.1, U5.5 (+): now also R15.2
- net +3V3_ISO renamed +4V5_ISO
- net +3V_Vref renamed +5V_Vref
- new net +5V_Ana: C17.1, C18.1, C35.1, C36.1, C41.1, C42.1, IC2.8 (VDD2), U4.8 (V+), U5.8 (V+)
- new net +5V_Cur_Sensor: C14.1, C15.1, C16.1, U3.13 (VDD)
Other:
- moved on the sheet: C36, C41, R19, U4C, U5C
