File: voltage_and_current_measurement.kicad_sch (KiCad schematic)
At the start: 88 parts, among them IC2 VIA2000SD, J6 V_bat_in, J7 V_bat_out, J8 V_bat_in, J9 V_bat_out, U3 ACS37030LLZATR-065B3, U4 CZ3A05, U5 OPA2328DR, U6 OPA2328DR

Commit message: Continue implementing ESP32 module
[KiCad Version: 10.0.3]
Parts:
- added R8: 18k, Resistor_SMD:R_0603_1608Metric_Pad0.98x0.95mm_HandSolder, symbol Device:R
- added U6: AMC1351DWV, Package_SO:SOIC-8_7.5x5.85mm_P1.27mm, symbol Isolator_Analog:AMC1351DWV
- C13: value 33p -> 100p
- IC2: now not fitted; now left out of the parts list
- R10: renamed from R9; value 12k -> 6.2k
- R9: renamed from R8; value 150k -> 18k
- renumbered D1 to D2, D2 to D3, D3 to D4, D4 to D5, R10 to R11, R11 to R12, R12 to R13, R13 to R14, R14 to R15, R15 to R16, R16 to R17, R17 to R18, R18 to R19, R19 to R20, R20 to R21, R21 to R22, R22 to R23, R23 to R24, U3 to U4, U4 to U5, U5 to U7, U6 to U8
Connections:
- net +4V5_ISO: now also U6.1 (VDD1); no longer IC2.1 (VDD1)
- net +5V_Ratiometric_Supply: now also U6.8 (VDD2); no longer IC2.8 (VDD2)
- net GND: now also U6.5 (GND2); no longer IC2.5 (GND2)
- net GND_ISO: now also U6.3 (GND1), U6.4 (GND1); no longer IC2.3 (SHTDN), IC2.4 (GND1)
- net V_bat_sense: now also R8.1; no longer R9.1
- net V_sig: now also U6.7 (OUTP); no longer IC2.7 (OUTP)
- net Vout_ref: now also U6.6 (OUTN); no longer IC2.6 (OUTN)
- net at C13.1, R10.1, R9.2: now also U6.2 (IN); no longer IC2.2 (VIN)
- new net: R8.2, R9.1
Other:
- note added: "RC Lowpass Resistor. 100 pF = 423 kHz (@-3dB)"
- note removed: "RC Lowpass Resistor. 33 pF = 423 kHz (@-3dB)"
- note removed: "TODO: ETSI PAREMPI YLI 75 dB SNR OPARI TÄHÄN... JOLLA ISOMPI LÄHTÖSWINGI"

Commit message: Add buffer OPA for Secondary battery measurement
[KiCad Version: 10.0.3]
Parts:
- renumbered C5 to C10, C6 to C11, C7 to C12, C8 to C13, C9 to C14, C10 to C15, C11 to C16, C12 to C17, C13 to C18, C14 to C19, C15 to C20, C16 to C21, C17 to C22, C18 to C23, C19 to C24, C20 to C25, C21 to C26, C22 to C27, C23 to C28, C24 to C29, C25 to C30, C26 to C31, C27 to C32, C28 to C33, C29 to C34, C30 to C35, C31 to C36, C32 to C37, C33 to C38, C34 to C39, C35 to C40, C36 to C41, C37 to C42, C38 to C43, C39 to C44, C40 to C45, C41 to C46, C42 to C47, C43 to C48, C44 to C49, C4 to C9, D2 to D4, D3 to D5, D4 to D6, D5 to D7, J6 to J3, J7 to J4, J8 to J5, J9 to J6, R8 to R22, R9 to R23, R10 to R24, R11 to R25, R12 to R26, R13 to R27, R14 to R28, R15 to R29, R16 to R30, R17 to R31, R18 to R32, R19 to R33, R20 to R34, R21 to R35, R22 to R36, R23 to R37, R24 to R38, U4 to U2, U5 to U3, U6 to U4, U7 to U5, U8 to U6

Commit message: Minor improvements. Add 3D model.
[KiCad Version: 10.0.4]
Parts:
- removed ACSVref1, ACSVref2, CurSig1, CurSig2: TestPoint, TestPoint:TestPoint_Pad_D1.0mm, symbol Connector:TestPoint
- removed C10, C9: 1000u, Capacitor_THT:C_Radial_D8.0mm_H11.5mm_P3.50mm, symbol Device:C
- removed C11, C12, C13: 1u, Capacitor_SMD:C_0603_1608Metric_Pad1.08x0.95mm_HandSolder, symbol Device:C
- removed D4, D5: 1.5SMCxxCA, Diode_SMD:D_SMC, symbol Diode:1.5SMCxxCA
- removed J3: V_bat_in, custom_footprints:AMASS_XT60PW-M_1x02_P7.20mm_Horizontal_with3DModel, symbol Connector:Conn_01x02_Pin
- removed J4: V_bat_out, custom_footprints:AMASS_XT60PW-M_1x02_P7.20mm_Horizontal_with3DModel, symbol Connector:Conn_01x02_Pin
- removed U2: ACS37030LLZATR-065B3, custom_footprints:ACS37030LLZATR-065B3, symbol Custom Symbols:ACS37032LLZATR-065B3
Other:
- note removed: "! MAX 100pF Load !"
- note removed: "ACS37030LLZATR-065B3 Sensitivity: 20.3 mV/A 65A = 1.32 V"
- note removed: "Current Measurement"
- note removed: "TARKASTA KUMPI ACS VERSIO ON TUO VREF / FAULT !!!!!!"
- moved on the sheet: C14, C15, C16, C17, C21, C22, C23, D6, D7, J5, J6, NT1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

Commit message: Fix Via offset.
[KiCad Version: 10.0.4]
Parts:
- removed C14, C15, C16, C17: 1000u, Capacitor_THT:C_Radial_D8.0mm_H11.5mm_P3.50mm, symbol Device:C
- removed J5: V_bat_in, custom_footprints:AMASS_XT60PW-M_1x02_P7.20mm_Horizontal_with3DModel, symbol Connector:Conn_01x02_Pin
- removed J6: V_bat_out, custom_footprints:AMASS_XT60PW-M_1x02_P7.20mm_Horizontal_with3DModel, symbol Connector:Conn_01x02_Pin
- removed U3: CZ3A05, CZ3A05, symbol SamacSys_Parts:CZ3A05
- added J3, J4: XT60PW-M, Connector_AMASS:AMASS_XT60PW-M_1x02_P7.20mm_Horizontal, symbol SamacSys_Parts:XT60PW-M
- added U3: CZ3723, custom_footprints:CZ3723, symbol Custom Symbols:CZ3723
- renumbered C18 to C12, C19 to C13, C20 to C14, C21 to C15, C22 to C16, C23 to C17, C24 to C18, C25 to C19, C26 to C20, C27 to C21, C28 to C22, C29 to C23, C30 to C24, C31 to C25, C32 to C26, C33 to C27, C34 to C28, C35 to C29, C36 to C30, C37 to C31, C38 to C32, C39 to C33, C40 to C34, C41 to C35, C42 to C36, C43 to C37, C44 to C38, C45 to C39, C46 to C40, C47 to C41, C48 to C42, C49 to C43, D6 to D4, D7 to D5, R22 to R23, R23 to R24, R24 to R25, R25 to R26, R26 to R27, R27 to R28, R28 to R29, R29 to R30, R30 to R31, R31 to R32, R32 to R33, R33 to R34, R34 to R35, R35 to R36, R36 to R37, R37 to R38, R38 to R39
Connections:
- net +5V_Ratiometric_Supply: now also U3.7 (VDD)
- net ACS_VREF: now also U3.5 (VREF)
- net GND: now also U3.10 (GND), U3.3 (GND), U3.4 (TEST1)
- net GND_ISO: now also J3.1, J3.3 (MH1), J3.4 (MH2), J4.1, J4.3 (MH1), J4.4 (MH2)
- net V_bat_in: now also J3.2, U3.1 (IP)
- net V_bat_out: now also J4.2, U3.2 (IN)
- net cur_sig: now also U3.6 (VOUT)
- no-connect marks 0 -> 2

Commit message: Minor improvements. Fix capacitor sizes.
[KiCad Version: 10.0.4]
Parts:
- C33: renamed from C32; footprint Capacitor_SMD:C_0603_1608Metric_Pad1.08x0.95mm_HandSolder -> Capacitor_SMD:C_0805_2012Metric_Pad1.18x1.45mm_HandSolder
- C34: renamed from C33; footprint Capacitor_SMD:C_0603_1608Metric_Pad1.08x0.95mm_HandSolder -> Capacitor_SMD:C_0805_2012Metric_Pad1.18x1.45mm_HandSolder
- C35: renamed from C34; footprint Capacitor_SMD:C_0603_1608Metric_Pad1.08x0.95mm_HandSolder -> Capacitor_SMD:C_0805_2012Metric_Pad1.18x1.45mm_HandSolder
- C36: renamed from C35; footprint Capacitor_SMD:C_0603_1608Metric_Pad1.08x0.95mm_HandSolder -> Capacitor_SMD:C_0805_2012Metric_Pad1.18x1.45mm_HandSolder
- renumbered C12 to C13, C13 to C14, C14 to C15, C15 to C16, C16 to C17, C17 to C18, C18 to C19, C19 to C20, C20 to C21, C21 to C22, C22 to C23, C23 to C24, C24 to C25, C25 to C26, C26 to C27, C27 to C28, C28 to C29, C29 to C30, C30 to C31, C31 to C32, C36 to C37, C37 to C38, C38 to C39, C39 to C40, C40 to C41, C41 to C42, C42 to C43, C43 to C44

Commit message: PCB improvements.
[KiCad Version: 10.0.4]
Parts:
- added GND1, TP1, TP2, TP3, TP4: TestPoint, TestPoint:TestPoint_Pad_D1.0mm, symbol Connector:TestPoint
- renumbered GND1 to GND2, GND2 to GND3, GND3 to GND4, GND4 to GND5
Connections:
- net ACS_VREF: now also TP3.1
- net GND_ISO: now also GND1.1
- net GND_bat_sense: now also TP2.1
- net V_bat_sense: now also TP1.1
- net cur_sig: now also TP4.1

Commit message: PCB Improvements.
[KiCad Version: 10.0.4]
Parts:
- removed IC2: VIA2000SD, SOIC127P1150X280-8N, symbol SamacSys_Parts:VIA2000SD
- renumbered J3 to J4, J4 to J5, TP1 to TP4, TP2 to TP5, TP3 to TP6, TP4 to TP7
Other:
- note removed: "TODO: VAIHDA TÄHÄN PAREMPI ANTURI..."
- moved on the sheet: C16, C17, C18, D4, D5, J4, J5, NT1, NT2, U3
