File: load_cell_measurement.kicad_sch (KiCad schematic)
At the start: 45 parts, among them IC4 MCP3564RT-E_ST, J10 Conn_01x04_Pin

Commit message: Commit before 5V rebase.
[KiCad Version: 10.0.4]
Parts:
- renumbered C85 to C100, C86 to C101, C87 to C102, C88 to C103, C89 to C104, C90 to C105, C91 to C106, C92 to C107, C93 to C108, C94 to C109, C95 to C110, C96 to C111, C97 to C112, C83 to C98, C84 to C99, I11 to I10, I10 to I11, J10 to J14

Commit message: Implemented SAR ADC Buffering on top layer with one OPA387
[KiCad Version: 10.0.4]
Parts:
- removed C106: 22u, Capacitor_SMD:C_1206_3216Metric_Pad1.33x1.80mm_HandSolder, symbol Device:C
- removed C110: 10u, Capacitor_SMD:C_0603_1608Metric_Pad1.08x0.95mm_HandSolder, symbol Device:C
- removed FB1: BLM21BD182SH1D, Inductor_SMD:L_0805_2012Metric_Pad1.15x1.40mm_HandSolder, symbol Device:FerriteBead
- removed I3: TestPoint, TestPoint:TestPoint_Pad_D1.0mm, symbol Connector:TestPoint
- removed R40: 1R, Resistor_SMD:R_0603_1608Metric_Pad0.98x0.95mm_HandSolder, symbol Device:R
- renumbered C98 to C106, C99 to C107, C100 to C108, C102 to C109, C103 to C110, C101 to C111, C104 to C112, C107 to C113, C108 to C114, C105 to C115, C109 to C116, C111 to C117, C112 to C118, I11 to I10, I4 to I3, I5 to I4, I6 to I5, I7 to I6, I8 to I7, I9 to I8, I10 to I9, J14 to J13, R37 to R38, R38 to R39, R36 to R40, R39 to R41, R41 to R42, R42 to R43, R43 to R44, R44 to R45, R45 to R46, R46 to R47, R47 to R48, R48 to R49
Connections:
- net +3V3_LC: now reaches C114.2, C116.2, IC4.4 (REFIN+/OUT), J13.4 (Pin_4)
- net +3V3_LC: now also C113.2, I3.1, IC4.1 (AVDD)
- net +3V3_Ana renamed +5V_Ana
- net +5V_Ana: no longer C113.2, I3.1, IC4.1 (AVDD)
Other:
- note added: "TODO: FIX R2 TO MATCH 5V SUPPLY AND 3V3 ADC INPUT !!!"
- note removed: "Dampening Snubber"
- note removed: "Ferrite is to block any noise from or to the Analog power plane. Load Cell will have long leads that may pick noise from the motors. It is not wanted that the noise gets injected to the analog supply."
- note removed: "Ferrite specs: Z = 1.8 kOhms I_max = 250 mA DC Resistance 500 mOhms"
- moved on the sheet: C109, C110, C113, C114, C116, C117, C118, IC4, J13, R38, R43, R44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

Commit message: Implemented dual SAR ADC Buffering and Current sensor ratiometric supply
[KiCad Version: 10.0.4]
Parts:
- renumbered C106 to C111, C107 to C112, C108 to C113, C109 to C114, C110 to C115, C111 to C116, C112 to C117, C113 to C118, C114 to C119, C115 to C120, C116 to C121, C117 to C122, C118 to C123, R38 to R41, R39 to R42, R40 to R43, R41 to R44, R42 to R45, R43 to R46, R44 to R47, R45 to R48, R46 to R49, R47 to R50, R48 to R51, R49 to R52

Commit message: Improved NTC measurements, improved layout. Added proper startup sequence for the power stages.
[KiCad Version: 10.0.4]
Parts:
- added R46, R48, R50: 10k, Resistor_SMD:R_0603_1608Metric_Pad0.98x0.95mm_HandSolder, symbol Device:R
- R47: renamed from R43; value 10k -> 18k
- R49: renamed from R44; value 10k -> 18k
- R51: renamed from R45; value 10k -> 18k
- renumbered C111 to C109, C112 to C110, C113 to C111, C114 to C112, C115 to C113, C116 to C114, C117 to C115, C118 to C116, C119 to C117, C121 to C118, C120 to C119, C122 to C120, C123 to C121, R41 to R44, R42 to R45, R46 to R52, R47 to R53, R48 to R54, R49 to R55, R50 to R56, R51 to R57, R52 to R58
Connections:
- net +5V_Ana: now also R46.2, R48.2, R50.2; no longer TH1.1, TH2.1, TH3.1
- net GND: now also TH1.2, TH2.2, TH3.2
- net NTC_1: now also TH1.1, R46.1; no longer TH1.2
- net NTC_2: now also TH2.1, R48.1; no longer TH2.2
- net NTC_3: now also TH3.1, R50.1; no longer TH3.2
Other:
- note added: "1uF & (NTC + 18k||10k) = RC Lowpass Filter ~ 25->500 Hz depending on NTC resistance."
- note added: "NTCG164BH103JT1: R-T Curve : 10kohm @25°C 200kohms @-40°C 300 ohms @150°C Voltage Swing: (10kohm/18kohm): 100 mV -> 3,159 V (-40°C/150°C)"
- note removed: "1uF & (NTC + 10k) = RC Lowpass Filter ~ 30->400 Hz depending on NTC resistance."
- note removed: "TODO: FIX R2 TO MATCH 5V SUPPLY AND 3V3 ADC INPUT !!!"
- moved on the sheet: C109, C110, C111, C114, C115, C119, R47, R49, R51, TH1, TH2, TH3
