File: load_cell_measurement.kicad_sch (KiCad schematic)
At the start: 43 parts, among them IC4 MCP3564RT-E_ST, J13 Conn_01x04_Pin

Commit message: Minor Tweaks.
[KiCad Version: 10.0.4]
Parts:
- renumbered C109 to C110, C110 to C111, C111 to C112, C112 to C113, C113 to C114, C114 to C115, C115 to C116, C116 to C117, C117 to C118, C118 to C119, C119 to C120, C120 to C121, C121 to C122

Commit message: Add Secondary battery voltage measurement. Minor tweaks.
[KiCad Version: 10.0.4]
Parts:
- renumbered C110 to C113, C111 to C114, C112 to C115, C113 to C116, C114 to C117, C115 to C118, C116 to C119, C117 to C120, C118 to C121, C119 to C122, C120 to C123, C121 to C124, C122 to C125, IC4 to IC5, R44 to R46, R45 to R47, R46 to R48, R47 to R49, R48 to R50, R49 to R51, R50 to R52, R51 to R53, R52 to R54, R53 to R55, R54 to R56, R55 to R57, R56 to R58, R57 to R59, R58 to R60

Commit message: Initial switch to ESP32 Module
[KiCad Version: 10.0.4]
Parts:
- renumbered C113 to C114, C114 to C115, C115 to C116, C116 to C117, C117 to C118, C118 to C119, C119 to C120, C120 to C121, C121 to C122, C122 to C123, C123 to C124, C124 to C125, C125 to C126

Commit message: Started implementing ESP32Module
[KiCad Version: 10.0.4]
Parts:
- renumbered J13 to J14
Changed lines of the file:
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@@
 		(in_pos_files yes)
 		(dnp no)
-		(property "Reference" "#PWR0200"
+		(property "Reference" "#PWR0202"
 			(at 76.2 105.41 0)
 			(hide yes)
@@
 			(project "motor_testbench_v1_0"
 				(path "/da638649-102c-44f9-b928-e91cd399cc2f/bd55160d-8c4c-42fa-b0ab-c795a19ea32a"
-					(reference "#PWR0200")
+					(reference "#PWR0202")
 					(unit 1)
 				)
@@
 		(in_pos_files yes)
 		(dnp no)
-		(property "Reference" "#PWR0196"
+		(property "Reference" "#PWR0198"
 			(at 44.45 173.99 0)
 			(hide yes)
@@
 			(project "motor_testbench_v1_0"
 				(path "/da638649-102c-44f9-b928-e91cd399cc2f/bd55160d-8c4c-42fa-b0ab-c795a19ea32a"
-					(reference "#PWR0196")
+					(reference "#PWR0198")
 					(unit 1)
 				)
@@
 		(in_pos_files yes)
 		(dnp no)
-		(property "Reference" "#PWR0220"
+		(property "Reference" "#PWR0222"
 			(at 185.42 80.01 0)
 			(hide yes)
@@
 			(project "motor_testbench_v1_0"
 				(path "/da638649-102c-44f9-b928-e91cd399cc2f/bd55160d-8c4c-42fa-b0ab-c795a19ea32a"
-					(reference "#PWR0220")
+					(reference "#PWR0222")
 					(unit 1)
 				)
@@
 		(in_pos_files yes)
 		(dnp no)
-		(property "Reference" "#PWR0218"
+		(property "Reference" "#PWR0220"
 			(at 149.86 173.99 0)
 			(hide yes)
@@
 			(project "motor_testbench_v1_0"
 				(path "/da638649-102c-44f9-b928-e91cd399cc2f/bd55160d-8c4c-42fa-b0ab-c795a19ea32a"
-					(reference "#PWR0218")
+					(reference "#PWR0220")
 					(unit 1)
 				)
@@
 		(in_pos_files yes)
 		(dnp no)
-		(property "Reference" "#PWR0201"
+		(property "Reference" "#PWR0203"
 			(at 76.2 118.11 0)
 			(hide yes)
@@
 			(project "motor_testbench_v1_0"
 				(path "/da638649-102c-44f9-b928-e91cd399cc2f/bd55160d-8c4c-42fa-b0ab-c795a19ea32a"
-					(reference "#PWR0201")
+					(reference "#PWR0203")
 					(unit 1)
 				)
@@
 		(in_pos_files yes)
 		(dnp no)
-		(property "Reference" "#PWR0211"
+		(property "Reference" "#PWR0213"
 			(at 124.46 45.72 0)
 			(hide yes)
@@
 			(project "motor_testbench_v1_0"
 				(path "/da638649-102c-44f9-b928-e91cd399cc2f/bd55160d-8c4c-42fa-b0ab-c795a19ea32a"
-					(reference "#PWR0211")
+					(reference "#PWR0213")
 					(unit 1)
 				)
@@
 		(in_pos_files yes)
 		(dnp no)
-		(property "Reference" "#PWR0204"
+		(property "Reference" "#PWR0206"
 			(at 97.79 173.99 0)
 			(hide yes)
@@
 			(project "motor_testbench_v1_0"
 				(path "/da638649-102c-44f9-b928-e91cd399cc2f/bd55160d-8c4c-42fa-b0ab-c795a19ea32a"
-					(reference "#PWR0204")
+					(reference "#PWR0206")
 					(unit 1)
 				)
@@
 		(in_pos_files yes)
 		(dnp no)
-		(property "Reference" "#PWR0208"
+		(property "Reference" "#PWR0210"
 			(at 118.11 93.98 0)
 			(hide yes)
@@
 			(project "motor_testbench_v1_0"
 				(path "/da638649-102c-44f9-b928-e91cd399cc2f/bd55160d-8c4c-42fa-b0ab-c795a19ea32a"
-					(reference "#PWR0208")
+					(reference "#PWR0210")
 					(unit 1)
 				)
@@
 		(in_pos_files yes)
 		(dnp no)
-		(property "Reference" "#PWR0222"
+		(property "Reference" "#PWR0224"
 			(at 191.77 95.25 0)
 			(hide yes)
@@
 			(project "motor_testbench_v1_0"
 				(path "/da638649-102c-44f9-b928-e91cd399cc2f/bd55160d-8c4c-42fa-b0ab-c795a19ea32a"
-					(reference "#PWR0222")
+					(reference "#PWR0224")
 					(unit 1)
 				)
@@
 		(in_pos_files yes)
 		(dnp no)
-		(property "Reference" "#PWR0197"
+		(property "Reference" "#PWR0199"
 			(at 54.61 173.9853 0)
 			(hide yes)
@@
 			(project "motor_testbench_v1_0"
 				(path "/da638649-102c-44f9-b928-e91cd399cc2f/bd55160d-8c4c-42fa-b0ab-c795a19ea32a"
-					(reference "#PWR0197")
+					(reference "#PWR0199")
 					(unit 1)
 				)
@@
 		(in_pos_files yes)
 		(dnp no)
-		(property "Reference" "#PWR0212"
+		(property "Reference" "#PWR0214"
 			(at 129.54 85.09 0)
 			(hide yes)
@@
 			(project "motor_testbench_v1_0"
 				(path "/da638649-102c-44f9-b928-e91cd399cc2f/bd55160d-8c4c-42fa-b0ab-c795a19ea32a"
-					(reference "#PWR0212")
+					(reference "#PWR0214")
 					(unit 1)
 				)
@@
 		(in_pos_files yes)
 		(dnp no)
-		(property "Reference" "#PWR0214"
+		(property "Reference" "#PWR0216"
 			(at 134.62 125.73 0)
 			(hide yes)
@@
 			(project "motor_testbench_v1_0"
 				(path "/da638649-102c-44f9-b928-e91cd399cc2f/bd55160d-8c4c-42fa-b0ab-c795a19ea32a"
-					(reference "#PWR0214")
+					(reference "#PWR0216")
 					(unit 1)
 				)
@@
 		(in_pos_files yes)
 		(dnp no)
-		(property "Reference" "#PWR0206"
+		(property "Reference" "#PWR0208"
 			(at 109.22 173.99 0)
 			(hide yes)
@@
 			(project "motor_testbench_v1_0"
 				(path "/da638649-102c-44f9-b928-e91cd399cc2f/bd55160d-8c4c-42fa-b0ab-c795a19ea32a"
-					(reference "#PWR0206")
+					(reference "#PWR0208")
 					(unit 1)
 				)
@@
 		(in_pos_files yes)
 		(dnp no)
-		(property "Reference" "#PWR0205"
+		(property "Reference" "#PWR0207"
 			(at 105.41 140.97 0)
 			(hide yes)
@@
 			(project "motor_testbench_v1_0"
 				(path "/da638649-102c-44f9-b928-e91cd399cc2f/bd55160d-8c4c-42fa-b0ab-c795a19ea32a"
-					(reference "#PWR0205")
+					(reference "#PWR0207")
 					(unit 1)
 				)
@@
 		(in_pos_files yes)
 		(dnp no)
-		(property "Reference" "#PWR0221"
+		(property "Reference" "#PWR0223"
 			(at 185.42 125.73 0)
 			(hide yes)
@@
 			(project "motor_testbench_v1_0"
 				(path "/da638649-102c-44f9-b928-e91cd399cc2f/bd55160d-8c4c-42fa-b0ab-c795a19ea32a"
-					(reference "#PWR0221")
+					(reference "#PWR0223")
 					(unit 1)
 				)
@@
 		(in_pos_files yes)
 		(dnp no)
-		(property "Reference" "J13"
+		(property "Reference" "J14"
 			(at 45.974 91.948 90)
 			(show_name no)
@@
 			(project "motor_testbench_v1_0"
 				(path "/da638649-102c-44f9-b928-e91cd399cc2f/bd55160d-8c4c-42fa-b0ab-c795a19ea32a"
-					(reference "J13")
+					(reference "J14")
 					(unit 1)
 				)
@@
 		(in_pos_files yes)
 		(dnp no)
-		(property "Reference" "#PWR0198"
+		(property "Reference" "#PWR0200"
 			(at 63.5 109.22 0)
 			(hide yes)
@@
 			(project "motor_testbench_v1_0"
 				(path "/da638649-102c-44f9-b928-e91cd399cc2f/bd55160d-8c4c-42fa-b0ab-c795a19ea32a"
-					(reference "#PWR0198")
+					(reference "#PWR0200")
 					(unit 1)
 				)
@@
 		(in_pos_files yes)
 		(dnp no)
-		(property "Reference" "#PWR0210"
+		(property "Reference" "#PWR0212"
 			(at 123.19 173.99 0)
 			(hide yes)
@@
 			(project "motor_testbench_v1_0"
 				(path "/da638649-102c-44f9-b928-e91cd399cc2f/bd55160d-8c4c-42fa-b0ab-c795a19ea32a"
-					(reference "#PWR0210")
+					(reference "#PWR0212")
 					(unit 1)
 				)
@@
 		(in_pos_files yes)
 		(dnp no)
-		(property "Reference" "#PWR0202"
+		(property "Reference" "#PWR0204"
 			(at 83.82 173.99 0)
 			(hide yes)
@@
 			(project "motor_testbench_v1_0"
 				(path "/da638649-102c-44f9-b928-e91cd399cc2f/bd55160d-8c4c-42fa-b0ab-c795a19ea32a"
-					(reference "#PWR0202")
+					(reference "#PWR0204")
 					(unit 1)
 				)
@@
 		(in_pos_files yes)
 		(dnp no)
-		(property "Reference" "#PWR0203"
+		(property "Reference" "#PWR0205"
 			(at 91.44 173.99 0)
 			(hide yes)
@@
 			(project "motor_testbench_v1_0"
 				(path "/da638649-102c-44f9-b928-e91cd399cc2f/bd55160d-8c4c-42fa-b0ab-c795a19ea32a"
-					(reference "#PWR0203")
+					(reference "#PWR0205")
 					(unit 1)
 				)
@@
 		(in_pos_files yes)
 		(dnp no)
-		(property "Reference" "#PWR0219"
+		(property "Reference" "#PWR0221"
 			(at 181.61 125.73 0)
 			(hide yes)
@@
 			(project "motor_testbench_v1_0"
 				(path "/da638649-102c-44f9-b928-e91cd399cc2f/bd55160d-8c4c-42fa-b0ab-c795a19ea32a"
-					(reference "#PWR0219")
+					(reference "#PWR0221")
 					(unit 1)
 				)
@@
 		(in_pos_files yes)
 		(dnp no)
-		(property "Reference" "#PWR0209"
+		(property "Reference" "#PWR0211"
 			(at 118.11 109.22 0)
 			(hide yes)
@@
 			(project "motor_testbench_v1_0"
 				(path "/da638649-102c-44f9-b928-e91cd399cc2f/bd55160d-8c4c-42fa-b0ab-c795a19ea32a"
-					(reference "#PWR0209")
+					(reference "#PWR0211")
 					(unit 1)
 				)
@@
 		(in_pos_files yes)
 		(dnp no)
-		(property "Reference" "#PWR0207"
+		(property "Reference" "#PWR0209"
 			(at 116.84 173.99 0)
 			(hide yes)
@@
 			(project "motor_testbench_v1_0"
 				(path "/da638649-102c-44f9-b928-e91cd399cc2f/bd55160d-8c4c-42fa-b0ab-c795a19ea32a"
-					(reference "#PWR0207")
+					(reference "#PWR0209")
 					(unit 1)
 				)
@@
 		(in_pos_files yes)
 		(dnp no)
-		(property "Reference" "#PWR0217"
+		(property "Reference" "#PWR0219"
 			(at 143.51 173.99 0)
 			(hide yes)
@@
 			(project "motor_testbench_v1_0"
 				(path "/da638649-102c-44f9-b928-e91cd399cc2f/bd55160d-8c4c-42fa-b0ab-c795a19ea32a"
-					(reference "#PWR0217")
+					(reference "#PWR0219")
 					(unit 1)
 				)
@@
 		(in_pos_files yes)
 		(dnp no)
-		(property "Reference" "#PWR0213"
+		(property "Reference" "#PWR0215"
 			(at 129.54 110.49 0)
 			(hide yes)
@@
 			(project "motor_testbench_v1_0"
 				(path "/da638649-102c-44f9-b928-e91cd399cc2f/bd55160d-8c4c-42fa-b0ab-c795a19ea32a"
-					(reference "#PWR0213")
+					(reference "#PWR0215")
 					(unit 1)
 				)
@@
 		(in_pos_files yes)
 		(dnp no)
-		(property "Reference" "#PWR0215"
+		(property "Reference" "#PWR0217"
 			(at 135.89 85.09 0)
 			(hide yes)
@@
 			(project "motor_testbench_v1_0"
 				(path "/da638649-102c-44f9-b928-e91cd399cc2f/bd55160d-8c4c-42fa-b0ab-c795a19ea32a"
-					(reference "#PWR0215")
+					(reference "#PWR0217")
 					(unit 1)
 				)
@@
 		(in_pos_files yes)
 		(dnp no)
-		(property "Reference" "#PWR0216"
+		(property "Reference" "#PWR0218"
 			(at 135.89 173.99 0)
 			(hide yes)
@@
 			(project "motor_testbench_v1_0"
 				(path "/da638649-102c-44f9-b928-e91cd399cc2f/bd55160d-8c4c-42fa-b0ab-c795a19ea32a"
-					(reference "#PWR0216")
+					(reference "#PWR0218")
 					(unit 1)
 				)
@@
 		(in_pos_files yes)
 		(dnp no)
-		(property "Reference" "#PWR0199"
+		(property "Reference" "#PWR0201"
 			(at 64.77 173.9853 0)
 			(hide yes)
@@
 			(project "motor_testbench_v1_0"
 				(path "/da638649-102c-44f9-b928-e91cd399cc2f/bd55160d-8c4c-42fa-b0ab-c795a19ea32a"
-					(reference "#PWR0199")
+					(reference "#PWR0201")
 					(unit 1)
 				)

Commit message: Continue implementing ESP32 module
[KiCad Version: 10.0.3]
Parts:
- removed R55, R58, R59, R60: 22R, Resistor_SMD:R_0603_1608Metric_Pad0.98x0.95mm_HandSolder, symbol Device:R
- removed R56: 0R, Resistor_SMD:R_0603_1608Metric_Pad0.98x0.95mm_HandSolder, symbol Device:R
- added C127: 1u, Capacitor_SMD:C_0603_1608Metric_Pad1.08x0.95mm_HandSolder, symbol Device:C
- added JP1, JP2: SolderJumper_2_Open, Jumper:SolderJumper-2_P1.3mm_Open_RoundedPad1.0x1.5mm, symbol Jumper:SolderJumper_2_Open
- added R62, R63: 10k, Resistor_SMD:R_0603_1608Metric_Pad0.98x0.95mm_HandSolder, symbol Device:R
- renumbered R46 to R47, R47 to R48, R48 to R49, R49 to R50, R50 to R51, R51 to R52, R52 to R53, R53 to R54, R54 to R55, R57 to R58
Connections:
- net +5V_Ana: now also C127.2, R63.2
- net DS_ADC_IRQ: now also I5.1, IC5.17 (~{IRQ}/MDAT), R55.1
- net DS_ADC_MCLK: now also I4.1, IC5.18 (MCLK)
- net DS_ADC_SPI_CS: now also I8.1, IC5.13 (~{CS})
- net DS_ADC_SPI_MOSI: now also I6.1, IC5.15 (SDI)
- net DS_ADC_SPI_SCLK: now also I7.1, IC5.14 (SCK)
- net GND: now also C127.1, JP2.2 (B), R62.1; no longer IC5.11 (CH6)
- new net: IC5.11 (CH6), JP1.1 (A), JP2.1 (A)
- new net: JP1.2 (B), R62.2, R63.1
Other:
- note added: "Default use: Connect JP1!"
- note added: "Possibility to add a 5V reference for the NTC measurements"
- note added: "This makes the measurement more Ratiometric / compensates variations in the 5V line."
- note removed: "TODO: LISÄÄ REDUNDANNTTIUS ELI HX711 VALMIUS HEADERILLA JA SOLDER BLOB I2C LIITÄNNÄLLÄ !!!!!"

Commit message: Add buffer OPA for Secondary battery measurement
[KiCad Version: 10.0.3]
Parts:
- removed I4: TestPoint, TestPoint:TestPoint_Pad_D1.0mm, symbol Connector:TestPoint
- renumbered C114 to C118, C115 to C119, C116 to C120, C117 to C121, C118 to C122, C119 to C123, C120 to C124, C121 to C125, C122 to C126, C123 to C127, C124 to C128, C125 to C129, C126 to C130, C127 to C131, J14 to J11, R47 to R61, R48 to R62, R49 to R63, R50 to R64, R51 to R65, R52 to R66, R53 to R67, R54 to R68, R55 to R69, R58 to R70, R62 to R71, R63 to R72
Connections:
- net DS_ADC_MCLK is gone; now on net GND: IC5.18 (MCLK)
Other:
- note added: "Default use: Bridge / Connect JP2!"
- note removed: "Default use: Connect JP1!"

Commit message: Minor improvements. Add 3D model.
[KiCad Version: 10.0.4]
Changed lines of the file:
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@@
 	(text "Load Cell ADC "
 		(exclude_from_sim no)
-		(at 204.47 38.608 0)
+		(at 251.968 36.576 0)
 		(effects
 			(font

Commit message: Fix Via offset.
[KiCad Version: 10.0.4]
Parts:
- renumbered C118 to C111, C119 to C112, C120 to C113, C121 to C114, C122 to C115, C123 to C116, C124 to C117, C125 to C118, C126 to C119, C127 to C120, C128 to C121, C129 to C122, C130 to C123, C131 to C124, I5 to I4, I6 to I5, I7 to I6, I8 to I7, I9 to I8, I10 to I9, IC5 to IC6, J11 to J9, JP1 to JP2, JP2 to JP3, R61 to R62, R62 to R63, R63 to R64, R64 to R65, R65 to R66, R66 to R67, R67 to R68, R68 to R69, R69 to R70, R70 to R71, R71 to R72, R72 to R73
