File: load_cell_measurement.kicad_sch (KiCad schematic)
At the start: 42 parts, among them IC6 MCP3564RT-E_ST, J9 Conn_01x04_Pin

Commit message: Minor improvements. Fix capacitor sizes.
[KiCad Version: 10.0.4]
Parts:
- C119: renamed from C118; footprint Capacitor_SMD:C_0603_1608Metric_Pad1.08x0.95mm_HandSolder -> Capacitor_SMD:C_0805_2012Metric_Pad1.18x1.45mm_HandSolder
- IC6: footprint SOP65P640X120-20N -> SamacSys_Parts:SOP65P640X120-20N
- renumbered C111 to C112, C112 to C113, C113 to C114, C114 to C115, C115 to C116, C116 to C117, C117 to C118, C119 to C120, C120 to C121, C121 to C122, C122 to C123, C123 to C124, C124 to C125, I8 to I4, I4 to TP2, I5 to TP3, I6 to TP4, I7 to TP5, I9 to TP6

Commit message: PCB improvements.
[KiCad Version: 10.0.4]
Parts:
- renumbered C112 to C113, C113 to C114, C114 to C115, C115 to C116, C116 to C117, C117 to C118, C118 to C119, C119 to C120, C120 to C121, C121 to C122, C122 to C123, C123 to C124, C124 to C125, C125 to C126, TP6 to TP10, TP2 to TP6, TP3 to TP7, TP4 to TP8, TP5 to TP9

Commit message: PCB Improvements.
[KiCad Version: 10.0.4]
Parts:
- renumbered J9 to J11, TP7 to TP10, TP8 to TP11, TP9 to TP12, TP10 to TP13, TP6 to TP9
