File: motor_testbench_v1_0.kicad_sch (KiCad schematic)
At the start: 30 parts, among them IC1 PJA3402_R1_00001, J1 Conn_01x05_Pin, J2 Conn_01x01_Pin, J3 Conn_01x01_Pin, J4 Conn_01x22_Pin, U1 ESP32-S3-DevKitC

Commit message: Initial switch to ESP32 Module
[KiCad Version: 10.0.4]
Parts:
- added U?: ESP32-S3-WROOM-2, RF_Module:ESP32-S3-WROOM-2, symbol RF_Module:ESP32-S3-WROOM-2
- renumbered J4 to J1, J1 to J2, J2 to J3, J3 to J4, R6 to R3, R7 to R4, R3 to R5, R4 to R6, R5 to R7
Connections:
- new net: U?.1 (GND), U?.40 (GND), U?.41 (GND)
Changed lines of the file:
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@@
 		(dnp no)
 		(fields_autoplaced yes)
-		(property "Reference" "#PWR011"
+		(property "Reference" "#PWR013"
 			(at 173.99 107.95 0)
 			(hide yes)
@@
 			(project "motor_testbench_v1_0"
 				(path "/da638649-102c-44f9-b928-e91cd399cc2f"
-					(reference "#PWR011")
+					(reference "#PWR013")
 					(unit 1)
 				)
@@
 		(dnp no)
 		(fields_autoplaced yes)
-		(property "Reference" "R7"
+		(property "Reference" "R4"
 			(at 129.54 71.1199 0)
 			(show_name no)
@@
 			(project "motor_testbench_v1_0"
 				(path "/da638649-102c-44f9-b928-e91cd399cc2f"
-					(reference "R7")
+					(reference "R4")
+					(unit 1)
+				)
+			)
+		)
+	)
+	(symbol
+		(lib_id "RF_Module:ESP32-S3-WROOM-2")
+		(at -20.32 128.27 0)
+		(unit 1)
+		(body_style 1)
+		(exclude_from_sim no)
+		(in_bom yes)
+		(on_board yes)
+		(in_pos_files yes)
+		(dnp no)
+		(fields_autoplaced yes)
+		(property "Reference" "U?"
+			(at -18.1767 77.47 0)
+			(show_name no)
+			(do_not_autoplace no)
+			(effects
+				(font
+					(size 1.27 1.27)
+				)
+				(justify left)
+			)
+		)
+		(property "Value" "ESP32-S3-WROOM-2"
+			(at -18.1767 80.01 0)
+			(show_name no)
+			(do_not_autoplace no)
+			(effects
+				(font
+					(size 1.27 1.27)
+				)
+				(justify left)
+			)
+		)
+		(property "Footprint" "RF_Module:ESP32-S3-WROOM-2"
+			(at -20.32 189.23 0)
+			(hide yes)
+			(show_name no)
+			(do_not_autoplace no)
+			(effects
+				(font
+					(size 1.27 1.27)
+				)
+			)
+		)
+		(property "Datasheet" "https://www.espressif.com/sites/default/files/documentation/esp32-s3-wroom-2_datasheet_en.pdf"
+			(at -20.32 191.77 0)
+			(hide yes)
+			(show_name no)
+			(do_not_autoplace no)
+			(effects
+				(font
+					(size 1.27 1.27)
+				)
+			)
+		)
+		(property "Description" "RF Module, 2.4 GHz, Wi­-Fi, Bluetooth, BLE, ESP32­-S3R8V"
+			(at -20.32 128.27 0)
+			(hide yes)
+			(show_name no)
+			(do_not_autoplace no)
+			(effects
+				(font
+					(size 1.27 1.27)
+				)
+			)
+		)
+		(pin "33"
+		)
+		(pin "34"
+		)
+		(pin "32"
+		)
+		(pin "35"
+		)
+		(pin "36"
+		)
+		(pin "25"
+		)
+		(pin "29"
+		)
+		(pin "30"
+		)
+		(pin "27"
+		)
+		(pin "31"
+		)
+		(pin "24"
+		)
+		(pin "26"
+		)
+		(pin "23"
+		)
+		(pin "28"
+		)
+		(pin "37"
+		)
+		(pin "39"
+		)
+		(pin "40"
+		)
+		(pin "38"
+		)
+		(pin "3"
+		)
+		(pin "7"
+		)
+		(pin "1"
+		)
+		(pin "2"
+		)
+		(pin "4"
+		)
+		(pin "5"
+		)
+		(pin "6"
+		)
+		(pin "8"
+		)
+		(pin "9"
+		)
+		(pin "10"
+		)
+		(pin "11"
+		)
+		(pin "12"
+		)
+		(pin "13"
+		)
+		(pin "14"
+		)
+		(pin "15"
+		)
+		(pin "16"
+		)
+		(pin "18"
+		)
+		(pin "19"
+		)
+		(pin "17"
+		)
+		(pin "20"
+		)
+		(pin "21"
+		)
+		(pin "22"
+		)
+		(pin "41"
+		)
+		(instances
+			(project "motor_testbench_v1_0"
+				(path "/da638649-102c-44f9-b928-e91cd399cc2f"
+					(reference "U?")
 					(unit 1)
 				)
@@
 		(in_pos_files yes)
 		(dnp no)
-		(property "Reference" "J1"
+		(property "Reference" "J2"
 			(at 171.45 58.42 90)
 			(show_name no)
@@
 			(project "motor_testbench_v1_0"
 				(path "/da638649-102c-44f9-b928-e91cd399cc2f"
-					(reference "J1")
+					(reference "J2")
 					(unit 1)
 				)
@@
 		(in_pos_files yes)
 		(dnp no)
-		(property "Reference" "R4"
+		(property "Reference" "R6"
 			(at 121.412 143.764 90)
 			(show_name no)
@@
 			(project "motor_testbench_v1_0"
 				(path "/da638649-102c-44f9-b928-e91cd399cc2f"
-					(reference "R4")
+					(reference "R6")
 					(unit 1)
 				)
@@
 		(in_pos_files yes)
 		(dnp no)
-		(property "Reference" "#PWR013"
+		(property "Reference" "#PWR015"
 			(at 199.39 85.09 0)
 			(hide yes)
@@
 			(project "motor_testbench_v1_0"
 				(path "/da638649-102c-44f9-b928-e91cd399cc2f"
-					(reference "#PWR013")
+					(reference "#PWR015")
 					(unit 1)
 				)
@@
 		(dnp no)
 		(fields_autoplaced yes)
-		(property "Reference" "J4"
+		(property "Reference" "J1"
 			(at 175.26 148.5899 0)
 			(show_name no)
@@
 			(project "motor_testbench_v1_0"
 				(path "/da638649-102c-44f9-b928-e91cd399cc2f"
-					(reference "J4")
+					(reference "J1")
 					(unit 1)
 				)
@@
 		(in_pos_files yes)
 		(dnp no)
-		(property "Reference" "#PWR0222"
+		(property "Reference" "#PWR011"
 			(at 151.13 185.42 0)
 			(hide yes)
@@
 			(project "motor_testbench_v1_0"
 				(path "/da638649-102c-44f9-b928-e91cd399cc2f"
-					(reference "#PWR0222")
+					(reference "#PWR011")
 					(unit 1)
 				)
@@
 		(in_pos_files yes)
 		(dnp no)
-		(property "Reference" "R5"
+		(property "Reference" "R7"
 			(at 121.412 148.844 90)
 			(show_name no)
@@
 			(project "motor_testbench_v1_0"
 				(path "/da638649-102c-44f9-b928-e91cd399cc2f"
-					(reference "R5")
+					(reference "R7")
 					(unit 1)
 				)
@@
 		(in_pos_files yes)
 		(dnp no)
-		(property "Reference" "#PWR012"
+		(property "Reference" "#PWR014"
 			(at 182.88 73.66 0)
 			(hide yes)
@@
 			(project "motor_testbench_v1_0"
 				(path "/da638649-102c-44f9-b928-e91cd399cc2f"
-					(reference "#PWR012")
+					(reference "#PWR014")
 					(unit 1)
 				)
@@
 		(in_pos_files yes)
 		(dnp no)
-		(property "Reference" "R3"
+		(property "Reference" "R5"
 			(at 121.412 141.224 90)
 			(show_name no)
@@
 			(project "motor_testbench_v1_0"
 				(path "/da638649-102c-44f9-b928-e91cd399cc2f"
-					(reference "R3")
+					(reference "R5")
 					(unit 1)
 				)
@@
 		(dnp no)
 		(fields_autoplaced yes)
-		(property "Reference" "#PWR010"
+		(property "Reference" "#PWR012"
 			(at 173.99 97.79 0)
 			(hide yes)
@@
 			(project "motor_testbench_v1_0"
 				(path "/da638649-102c-44f9-b928-e91cd399cc2f"
-					(reference "#PWR010")
+					(reference "#PWR012")
 					(unit 1)
 				)
@@
 		(in_pos_files yes)
 		(dnp no)
-		(property "Reference" "J2"
+		(property "Reference" "J3"
 			(at 185.166 67.056 0)
 			(show_name no)
@@
 			(project "motor_testbench_v1_0"
 				(path "/da638649-102c-44f9-b928-e91cd399cc2f"
-					(reference "J2")
+					(reference "J3")
 					(unit 1)
 				)
@@
 		(dnp no)
 		(fields_autoplaced yes)
-		(property "Reference" "R6"
+		(property "Reference" "R3"
 			(at 129.54 60.9599 0)
 			(show_name no)
@@
 			(project "motor_testbench_v1_0"
 				(path "/da638649-102c-44f9-b928-e91cd399cc2f"
-					(reference "R6")
+					(reference "R3")
 					(unit 1)
 				)
@@
 		(in_pos_files yes)
 		(dnp no)
-		(property "Reference" "#PWR0220"
+		(property "Reference" "#PWR010"
 			(at 151.13 132.08 0)
 			(hide yes)
@@
 			(project "motor_testbench_v1_0"
 				(path "/da638649-102c-44f9-b928-e91cd399cc2f"
-					(reference "#PWR0220")
+					(reference "#PWR010")
 					(unit 1)
 				)
@@
 		(in_pos_files yes)
 		(dnp no)
-		(property "Reference" "J3"
+		(property "Reference" "J4"
 			(at 185.166 74.676 0)
 			(show_name no)
@@
 			(project "motor_testbench_v1_0"
 				(path "/da638649-102c-44f9-b928-e91cd399cc2f"
-					(reference "J3")
+					(reference "J4")
 					(unit 1)
 				)

Commit message: Commit before complete rework for ESP32S3Module
[KiCad Version: 10.0.4]
Parts:
- added J?: USB_C_Receptacle_USB2.0_16P, Connector_USB:USB_C_Receptacle_GCT_USB4105-xx-A_16P_TopMnt_Horizontal, symbol Connector:USB_C_Receptacle_USB2.0_16P
- gave numbers to parts that had none: 1
- renumbered U1 to U2
Connections:
- net +3V3_ESP: now also U1.2 (3V3)
- net DS_ADC_SPI_MISO: now also U1.7 (IO7)
- net DS_ADC_SPI_SCLK: now also U1.6 (IO6)
- net ESP_GPIO0: now also U1.27 (IO0)
- net ESP_GPIO1: now also U1.39 (IO1)
- net ESP_GPIO10: now also U1.18 (IO10)
- net ESP_GPIO11: now also U1.19 (IO11)
- net ESP_GPIO12: now also U1.20 (IO12)
- net ESP_GPIO14: now also U1.22 (IO14)
- net ESP_GPIO2: now also U1.38 (IO2)
- net ESP_GPIO3: now also U1.15 (IO3)
- net ESP_GPIO39: now also U1.32 (MTCK/IO39)
- net ESP_GPIO40: now also U1.33 (MTDO/IO40)
- net ESP_GPIO41: now also U1.34 (MTDI/IO41)
- net ESP_GPIO42: now also U1.35 (MTMS/IO42)
- net ESP_GPIO45: now also U1.26 (IO45)
- net ESP_GPIO46: now also U1.16 (IO46)
- net ESP_GPIO47: now also U1.24 (IO47)
- net ESP_GPIO48: now also U1.25 (IO48)
- net ESP_GPIO8: now also U1.12 (IO8)
- net ESP_GPIO9: now also U1.17 (IO9)
- net FAN_PWM: now also U1.4 (IO4)
- net GND: now also U1.1 (GND), U1.40 (GND), U1.41 (GND)
- net MISO: now also U1.21 (IO13)
- net V_secondary_Bat: now also U1.5 (IO5)
- new net: J?.A1 (GND), J?.A12 (GND), J?.B1 (GND), J?.B12 (GND)
- new net: J?.A4 (VBUS), J?.A9 (VBUS), J?.B4 (VBUS), J?.B9 (VBUS)
Other:
- moved on the sheet: U1

Commit message: Started implementing ESP32Module
[KiCad Version: 10.0.4]
Parts:
- J1: renamed from J?; footprint Connector_USB:USB_C_Receptacle_GCT_USB4105-xx-A_16P_TopMnt_Horizontal -> Connector_USB:USB_C_Receptacle_HCTL_HC-TYPE-C-16P-01A
- renumbered J1 to J2, J2 to J3, J3 to J4, J4 to J5
Changed lines of the file:
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@@
 		(dnp no)
 		(fields_autoplaced yes)
-		(property "Reference" "#PWR013"
+		(property "Reference" "#PWR015"
 			(at 173.99 107.95 0)
 			(hide yes)
@@
 			(project "motor_testbench_v1_0"
 				(path "/da638649-102c-44f9-b928-e91cd399cc2f"
-					(reference "#PWR013")
+					(reference "#PWR015")
 					(unit 1)
 				)
@@
 		(in_pos_files yes)
 		(dnp no)
-		(property "Reference" "#PWR01"
+		(property "Reference" "#PWR03"
 			(at 77.47 191.77 0)
 			(hide yes)
@@
 			(project "motor_testbench_v1_0"
 				(path "/da638649-102c-44f9-b928-e91cd399cc2f"
-					(reference "#PWR01")
+					(reference "#PWR03")
 					(unit 1)
 				)
@@
 		(in_pos_files yes)
 		(dnp no)
-		(property "Reference" "#PWR0223"
+		(property "Reference" "#PWR01"
 			(at -17.78 91.44 0)
 			(hide yes)
@@
 			(project "motor_testbench_v1_0"
 				(path "/da638649-102c-44f9-b928-e91cd399cc2f"
-					(reference "#PWR0223")
+					(reference "#PWR01")
 					(unit 1)
 				)
@@
 		(dnp no)
 		(fields_autoplaced yes)
-		(property "Reference" "#PWR09"
+		(property "Reference" "#PWR011"
 			(at 135.89 85.09 0)
 			(hide yes)
@@
 			(project "motor_testbench_v1_0"
 				(path "/da638649-102c-44f9-b928-e91cd399cc2f"
-					(reference "#PWR09")
+					(reference "#PWR011")
 					(unit 1)
 				)
@@
 		(in_pos_files yes)
 		(dnp no)
-		(property "Reference" "J2"
+		(property "Reference" "J3"
 			(at 171.45 58.42 90)
 			(show_name no)
@@
 			(project "motor_testbench_v1_0"
 				(path "/da638649-102c-44f9-b928-e91cd399cc2f"
-					(reference "J2")
+					(reference "J3")
 					(unit 1)
 				)
@@
 		(in_pos_files yes)
 		(dnp no)
-		(property "Reference" "#PWR0224"
+		(property "Reference" "#PWR02"
 			(at -17.78 190.5 0)
 			(hide yes)
@@
 			(project "motor_testbench_v1_0"
 				(path "/da638649-102c-44f9-b928-e91cd399cc2f"
-					(reference "#PWR0224")
+					(reference "#PWR02")
 					(unit 1)
 				)
@@
 		(in_pos_files yes)
 		(dnp no)
-		(property "Reference" "#PWR015"
+		(property "Reference" "#PWR017"
 			(at 199.39 85.09 0)
 			(hide yes)
@@
 			(project "motor_testbench_v1_0"
 				(path "/da638649-102c-44f9-b928-e91cd399cc2f"
-					(reference "#PWR015")
+					(reference "#PWR017")
 					(unit 1)
 				)
@@
 		(dnp no)
 		(fields_autoplaced yes)
-		(property "Reference" "#PWR05"
+		(property "Reference" "#PWR07"
 			(at 81.28 96.52 0)
 			(hide yes)
@@
 			(project "motor_testbench_v1_0"
 				(path "/da638649-102c-44f9-b928-e91cd399cc2f"
-					(reference "#PWR05")
+					(reference "#PWR07")
 					(unit 1)
 				)
@@
 		(dnp no)
 		(fields_autoplaced yes)
-		(property "Reference" "J1"
+		(property "Reference" "J2"
 			(at 175.26 148.5899 0)
 			(show_name no)
@@
 			(project "motor_testbench_v1_0"
 				(path "/da638649-102c-44f9-b928-e91cd399cc2f"
-					(reference "J1")
+					(reference "J2")
 					(unit 1)
 				)
@@
 		(in_pos_files yes)
 		(dnp no)
-		(property "Reference" "#PWR04"
+		(property "Reference" "#PWR06"
 			(at 78.74 78.74 0)
 			(hide yes)
@@
 			(project "motor_testbench_v1_0"
 				(path "/da638649-102c-44f9-b928-e91cd399cc2f"
-					(reference "#PWR04")
+					(reference "#PWR06")
 					(unit 1)
 				)
@@
 		(in_pos_files yes)
 		(dnp no)
-		(property "Reference" "#PWR011"
+		(property "Reference" "#PWR013"
 			(at 151.13 185.42 0)
 			(hide yes)
@@
 			(project "motor_testbench_v1_0"
 				(path "/da638649-102c-44f9-b928-e91cd399cc2f"
-					(reference "#PWR011")
+					(reference "#PWR013")
 					(unit 1)
 				)
@@
 		(dnp no)
 		(fields_autoplaced yes)
-		(property "Reference" "#PWR03"
+		(property "Reference" "#PWR05"
 			(at 78.74 64.77 0)
 			(hide yes)
@@
 			(project "motor_testbench_v1_0"
 				(path "/da638649-102c-44f9-b928-e91cd399cc2f"
-					(reference "#PWR03")
+					(reference "#PWR05")
 					(unit 1)
 				)
@@
 		(in_pos_files yes)
 		(dnp no)
-		(property "Reference" "#PWR014"
+		(property "Reference" "#PWR016"
 			(at 182.88 73.66 0)
 			(hide yes)
@@
 			(project "motor_testbench_v1_0"
 				(path "/da638649-102c-44f9-b928-e91cd399cc2f"
-					(reference "#PWR014")
+					(reference "#PWR016")
 					(unit 1)
 				)
@@
 		(in_pos_files yes)
 		(dnp no)
-		(property "Reference" "#PWR07"
+		(property "Reference" "#PWR09"
 			(at 125.73 59.69 0)
 			(hide yes)
@@
 			(project "motor_testbench_v1_0"
 				(path "/da638649-102c-44f9-b928-e91cd399cc2f"
-					(reference "#PWR07")
+					(reference "#PWR09")
 					(unit 1)
 				)
@@
 		(in_pos_files yes)
 		(dnp no)
-		(property "Reference" "#PWR02"
+		(property "Reference" "#PWR04"
 			(at 78.74 33.02 0)
 			(hide yes)
@@
 			(project "motor_testbench_v1_0"
 				(path "/da638649-102c-44f9-b928-e91cd399cc2f"
-					(reference "#PWR02")
+					(reference "#PWR04")
 					(unit 1)
 				)
@@
 		(dnp no)
 		(fields_autoplaced yes)
-		(property "Reference" "#PWR012"
+		(property "Reference" "#PWR014"
 			(at 173.99 97.79 0)
 			(hide yes)
@@
 			(project "motor_testbench_v1_0"
 				(path "/da638649-102c-44f9-b928-e91cd399cc2f"
-					(reference "#PWR012")
+					(reference "#PWR014")
 					(unit 1)
 				)
@@
 		(dnp no)
 		(fields_autoplaced yes)
-		(property "Reference" "J?"
+		(property "Reference" "J1"
 			(at -62.23 121.92 0)
 			(show_name no)
@@
 			)
 		)
-		(property "Footprint" "Connector_USB:USB_C_Receptacle_GCT_USB4105-xx-A_16P_TopMnt_Horizontal"
+		(property "Footprint" "Connector_USB:USB_C_Receptacle_HCTL_HC-TYPE-C-16P-01A"
 			(at -58.42 144.78 0)
 			(hide yes)
@@
 			(project "motor_testbench_v1_0"
 				(path "/da638649-102c-44f9-b928-e91cd399cc2f"
-					(reference "J?")
+					(reference "J1")
 					(unit 1)
 				)
@@
 		(in_pos_files yes)
 		(dnp no)
-		(property "Reference" "J3"
+		(property "Reference" "J4"
 			(at 185.166 67.056 0)
 			(show_name no)
@@
 			(project "motor_testbench_v1_0"
 				(path "/da638649-102c-44f9-b928-e91cd399cc2f"
-					(reference "J3")
+					(reference "J4")
 					(unit 1)
 				)
@@
 		(dnp no)
 		(fields_autoplaced yes)
-		(property "Reference" "#PWR06"
+		(property "Reference" "#PWR08"
 			(at 88.9 96.52 0)
 			(hide yes)
@@
 			(project "motor_testbench_v1_0"
 				(path "/da638649-102c-44f9-b928-e91cd399cc2f"
-					(reference "#PWR06")
+					(reference "#PWR08")
 					(unit 1)
 				)
@@
 		(in_pos_files yes)
 		(dnp no)
-		(property "Reference" "#PWR010"
+		(property "Reference" "#PWR012"
 			(at 151.13 132.08 0)
 			(hide yes)
@@
 			(project "motor_testbench_v1_0"
 				(path "/da638649-102c-44f9-b928-e91cd399cc2f"
-					(reference "#PWR010")
+					(reference "#PWR012")
 					(unit 1)
 				)
@@
 		(in_pos_files yes)
 		(dnp no)
-		(property "Reference" "J4"
+		(property "Reference" "J5"
 			(at 185.166 74.676 0)
 			(show_name no)
@@
 			(project "motor_testbench_v1_0"
 				(path "/da638649-102c-44f9-b928-e91cd399cc2f"
-					(reference "J4")
+					(reference "J5")
 					(unit 1)
 				)
@@
 		(exclude_from_sim no)
 		(in_bom no)
-		(on_board yes)
+		(on_board no)
 		(in_pos_files yes)
 		(dnp no)
@@
 		(dnp no)
 		(fields_autoplaced yes)
-		(property "Reference" "#PWR08"
+		(property "Reference" "#PWR010"
 			(at 125.73 85.09 0)
 			(hide yes)
@@
 			(project "motor_testbench_v1_0"
 				(path "/da638649-102c-44f9-b928-e91cd399cc2f"
-					(reference "#PWR08")
+					(reference "#PWR010")
 					(unit 1)
 				)
