File: power_regulation.kicad_sch (KiCad schematic)
At the start: 120 parts, among them IC3 NCV8184DR2G, IC4 MIE1W0505BGLVH-3R-P, J10 Conn_01x02_Pin, J11 Conn_01x02_Pin, J12 Conn_01x02_Pin, J9 V_bat_secondary, U10 TPS7A2055PDBVR, U11 TLV75733PDYDR, U12 TPS7A2050PDBVR, U13 TPS7A2033PDBVR, U14 TPS7A2018PDBVRG4, U15 TPS7A2050PDBVR, U16 TPS7A2050PDBVR, U17 TPS7A2033PDBVR, U18 TPS7A2045PDBVR, U6 MCP1502T-50E/CHY, U7 TPS62933, U8 TPS62933, U9 OPA2387DR

Commit message: Add full ESP32 DevKit Length PCB.
[KiCad Version: 10.0.4]
Parts:
- C54: footprint Capacitor_THT:CP_Radial_D6.3mm_P2.50mm -> Capacitor_SMD:CP_Elec_6.3x5.3
- D6: footprint Diode_SMD:D_SMA_Handsoldering -> Diode_SMD:D_SMA
Changed lines of the file:
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@@
 			)
 		)
-		(property "Footprint" "Diode_SMD:D_SMA_Handsoldering"
+		(property "Footprint" "Diode_SMD:D_SMA"
 			(at 130.81 38.1 0)
 			(hide yes)
@@
 			)
 		)
-		(property "Footprint" "Capacitor_THT:CP_Radial_D6.3mm_P2.50mm"
+		(property "Footprint" "Capacitor_SMD:CP_Elec_6.3x5.3"
 			(at 78.4352 248.92 0)
 			(hide yes)

Commit message: Initial switch to ESP32 Module
[KiCad Version: 10.0.4]
Parts:
- added C73: 1u, Capacitor_SMD:C_0603_1608Metric_Pad1.08x0.95mm_HandSolder, symbol Device:C
- renumbered C99 to C100, C100 to C101, C101 to C102, C102 to C103, C103 to C104, C104 to C105, C105 to C106, C106 to C107, C107 to C108, C108 to C109, C109 to C110, C110 to C111, C111 to C112, C112 to C113, C71 to C70, C70 to C71, C73 to C74, C74 to C75, C75 to C76, C76 to C77, C77 to C78, C78 to C79, C79 to C80, C80 to C81, C81 to C82, C82 to C83, C83 to C84, C84 to C85, C85 to C86, C86 to C87, C87 to C88, C88 to C89, C89 to C90, C90 to C91, C91 to C92, C92 to C93, C93 to C94, C94 to C95, C95 to C96, C96 to C97, C97 to C98, C98 to C99
Connections:
- net +6V_Buck_Out: now also C73.2
- net GND: now also C73.1
Other:
- note added: "TODO: TOTEUTA ANTUREIDEN POWER SEQUENCE !!!!"
- moved on the sheet: C45, C70, C87, C95, C97, R24, U14

Commit message: Commit before complete rework for ESP32S3Module
[KiCad Version: 10.0.4]
Parts:
- renumbered C101 to C100, C102 to C101, C103 to C102, C104 to C103, C105 to C104, C106 to C105, C107 to C106, C108 to C107, C109 to C108, C110 to C109, C111 to C110, C112 to C111, C113 to C112, C45 to C113, C46 to C45, C47 to C46, C48 to C47, C49 to C48, C50 to C49, C51 to C50, C52 to C51, C53 to C52, C54 to C53, C55 to C54, C56 to C55, C57 to C56, C58 to C57, C59 to C58, C60 to C59, C61 to C60, C62 to C61, C63 to C62, C64 to C63, C65 to C64, C66 to C65, C67 to C66, C68 to C67, C69 to C68, C70 to C69, C71 to C70, C72 to C71, C73 to C72, C74 to C73, C75 to C74, C76 to C75, C77 to C76, C78 to C77, C79 to C78, C80 to C79, C81 to C80, C82 to C81, C83 to C82, C84 to C83, C85 to C84, C86 to C85, C87 to C86, C88 to C87, C89 to C88, C90 to C89, C91 to C90, C92 to C91, C93 to C92, C94 to C93, C95 to C94, C96 to C95, C98 to C96, C99 to C98, C100 to C99, R25 to R24, R26 to R25, R27 to R26, R28 to R27, R29 to R28, R30 to R29, R31 to R30, R32 to R31, R33 to R32, R34 to R33, R35 to R34, R36 to R35, R37 to R36, R38 to R37, R39 to R38, R40 to R39, R41 to R40, R42 to R41, R43 to R42, R44 to R43, R45 to R44, R24 to R45, U9 to U10, U10 to U11, U11 to U12, U12 to U13, U13 to U14, U14 to U15, U15 to U16, U16 to U17, U17 to U18, U18 to U19, U6 to U7, U7 to U8, U8 to U9

Commit message: Started implementing ESP32Module
[KiCad Version: 10.0.4]
Parts:
- removed D5: 1.5SMCxxCA, Diode_SMD:D_SMC, symbol Diode:1.5SMCxxCA
- added D?: ESDA5V3L, Package_TO_SOT_SMD:SOT-23-3, symbol Power_Protection:ESDA5V3L
- renumbered J9 to J10, J10 to J11, J11 to J12, J12 to J13
Connections:
- net +VBat_Secondary: now also D?.1 (K), D?.2 (K)
- net GND: now also D?.3 (A)
Other:
- note added: "TODO: VAIHDA TÄHÄN Mouser No: 637-PSOT36 Mfr. No: PSOT36"
- moved on the sheet: J10

Commit message: Add few todo's
[KiCad Version: 10.0.4]
Parts:
- gave numbers to parts that had none: 1
Other:
- note added: "Startup-sequence (chronological order from top to bottom): 1. Battery Starts: +6V_Buck -> +5V5_bus (Always On with Battery) 2. 5V5_bus Starts: MCP1502, +1V8_AVDD and +3V3_DIO 3. 3V3_DIO Starts: ESP32 3. 1V8_AVDD Starts: +5V_Ana. 4. +5V_Ana Starts: OPA2387's, NCV8184 5. NCV8184 Starts: Current Sensor, Isolating OpAmp KORJAA TUO NCV STARTUP SEKVENSSI !!!!!!!!!"
- note removed: "Startup-sequence (chronological order from top to bottom): 1. Battery Starts: +6V_Buck -> +5V5_bus (Always On with Battery) 2. 5V5_bus Starts: MCP1502, +1V8_AVDD and +3V3_DIO 3. 3V3_DIO Starts: ESP32 3. 1V8_AVDD Starts: +5V_Ana. 4. +5V_Ana Starts: OPA2387's, NCV8184 5. NCV8184 Starts: Current Sensor, Isolating OpAmp"
- moved on the sheet: C113, R45
Changed lines of the file:
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@@
 		)
 	)
-	(text "Startup-sequence (chronological order from top to bottom):\n1. Battery  Starts: +6V_Buck -> +5V5_bus (Always On with Battery) \n2. 5V5_bus  Starts: MCP1502, +1V8_AVDD and +3V3_DIO\n3. 3V3_DIO  Starts: ESP32\n3. 1V8_AVDD Starts: +5V_Ana.\n4. +5V_Ana  Starts: OPA2387's, NCV8184\n5. NCV8184  Starts: Current Sensor, Isolating OpAmp"
+	(text "Startup-sequence (chronological order from top to bottom):\n1. Battery  Starts: +6V_Buck -> +5V5_bus (Always On with Battery) \n2. 5V5_bus  Starts: MCP1502, +1V8_AVDD and +3V3_DIO\n3. 3V3_DIO  Starts: ESP32\n3. 1V8_AVDD Starts: +5V_Ana.\n4. +5V_Ana  Starts: OPA2387's, NCV8184\n5. NCV8184  Starts: Current Sensor, Isolating OpAmp\n\nKORJAA TUO NCV STARTUP SEKVENSSI !!!!!!!!!"
 		(exclude_from_sim no)
-		(at 123.19 -28.448 0)
+		(at 124.714 -33.782 0)
 		(effects
 			(font
@@
 	(text "TODO: TOTEUTA ANTUREIDEN POWER SEQUENCE !!!!"
 		(exclude_from_sim no)
-		(at 450.088 176.022 0)
+		(at 366.268 -14.478 0)
 		(effects
 			(font
@@
 	)
 	(junction
-		(at 449.58 162.56)
+		(at 365.76 -27.94)
 		(diameter 0)
 		(color 0 0 0 0)
@@
 	(wire
 		(pts
-			(xy 449.58 153.67) (xy 449.58 162.56)
+			(xy 365.76 -36.83) (xy 365.76 -27.94)
 		)
 		(stroke
@@
 	(wire
 		(pts
-			(xy 449.58 144.78) (xy 449.58 146.05)
+			(xy 365.76 -45.72) (xy 365.76 -44.45)
 		)
 		(stroke
@@
 	(wire
 		(pts
-			(xy 449.58 162.56) (xy 455.93 162.56)
+			(xy 365.76 -27.94) (xy 372.11 -27.94)
 		)
 		(stroke
@@
 		(in_pos_files yes)
 		(dnp no)
-		(property "Reference" "D?"
+		(property "Reference" "D5"
 			(at 58.674 251.968 0)
 			(show_name no)
@@
 			(project "motor_testbench_v1_0"
 				(path "/da638649-102c-44f9-b928-e91cd399cc2f/f4ebbd2c-ae23-469d-a040-5f643f36c41b"
-					(reference "D?")
+					(reference "D5")
 					(unit 1)
 				)
@@
 		(dnp no)
 		(fields_autoplaced yes)
-		(property "Reference" "#PWR081"
+		(property "Reference" "#PWR082"
 			(at 54.61 49.53 0)
 			(hide yes)
@@
 			(project "motor_testbench_v1_0"
 				(path "/da638649-102c-44f9-b928-e91cd399cc2f/f4ebbd2c-ae23-469d-a040-5f643f36c41b"
-					(reference "#PWR081")
+					(reference "#PWR082")
 					(unit 1)
 				)
@@
 	(symbol
 		(lib_id "power:GND")
-		(at 449.58 170.18 0)
+		(at 365.76 -20.32 0)
 		(unit 1)
 		(body_style 1)
@@
 		(dnp no)
 		(property "Reference" "#PWR0197"
-			(at 449.58 176.53 0)
+			(at 365.76 -13.97 0)
 			(hide yes)
 			(show_name no)
@@
 		)
 		(property "Value" "GND"
-			(at 449.326 174.498 0)
+			(at 365.506 -16.002 0)
 			(hide yes)
 			(show_name no)
@@
 		)
 		(property "Footprint" ""
-			(at 449.58 170.18 0)
+			(at 365.76 -20.32 0)
 			(hide yes)
 			(show_name no)
@@
 		)
 		(property "Datasheet" ""
-			(at 449.58 170.18 0)
+			(at 365.76 -20.32 0)
 			(hide yes)
 			(show_name no)
@@
 		)
 		(property "Description" "Power symbol creates a global label with name \"GND\" , ground"
-			(at 449.58 170.18 0)
+			(at 365.76 -20.32 0)
 			(hide yes)
 			(show_name no)
@@
 	(symbol
 		(lib_id "power:+3V3")
-		(at 449.58 144.78 0)
+		(at 365.76 -45.72 0)
 		(unit 1)
 		(body_style 1)
@@
 		(dnp no)
 		(property "Reference" "#PWR0196"
-			(at 449.58 148.59 0)
+			(at 365.76 -41.91 0)
 			(hide yes)
 			(show_name no)
@@
 		)
 		(property "Value" "+5V_Ana"
-			(at 454.914 143.256 0)
+			(at 371.094 -47.244 0)
 			(show_name no)
 			(do_not_autoplace no)
@@
 		)
 		(property "Footprint" ""
-			(at 449.58 144.78 0)
+			(at 365.76 -45.72 0)
 			(hide yes)
 			(show_name no)
@@
 		)
 		(property "Datasheet" ""
-			(at 449.58 144.78 0)
+			(at 365.76 -45.72 0)
 			(hide yes)
 			(show_name no)
@@
 		)
 		(property "Description" "Power symbol creates a global label with name \"+3V3\""
-			(at 449.58 144.78 0)
+			(at 365.76 -45.72 0)
 			(hide yes)
 			(show_name no)
@@
 		(in_pos_files yes)
 		(dnp no)
-		(property "Reference" "#PWR082"
+		(property "Reference" "#PWR083"
 			(at 54.61 172.72 0)
 			(hide yes)
@@
 			(project "motor_testbench_v1_0"
 				(path "/da638649-102c-44f9-b928-e91cd399cc2f/f4ebbd2c-ae23-469d-a040-5f643f36c41b"
-					(reference "#PWR082")
+					(reference "#PWR083")
 					(unit 1)
 				)
@@
 		(dnp no)
 		(fields_autoplaced yes)
-		(property "Reference" "#PWR086"
+		(property "Reference" "#PWR087"
 			(at 62.23 66.04 0)
 			(hide yes)
@@
 			(project "motor_testbench_v1_0"
 				(path "/da638649-102c-44f9-b928-e91cd399cc2f/f4ebbd2c-ae23-469d-a040-5f643f36c41b"
-					(reference "#PWR086")
+					(reference "#PWR087")
 					(unit 1)
 				)
@@
 		(dnp no)
 		(fields_autoplaced yes)
-		(property "Reference" "#PWR087"
+		(property "Reference" "#PWR081"
 			(at 52.07 257.81 0)
 			(hide yes)
@@
 			(project "motor_testbench_v1_0"
 				(path "/da638649-102c-44f9-b928-e91cd399cc2f/f4ebbd2c-ae23-469d-a040-5f643f36c41b"
-					(reference "#PWR087")
+					(reference "#PWR081")
 					(unit 1)
 				)
@@
 		(dnp no)
 		(fields_autoplaced yes)
-		(property "Reference" "#PWR083"
+		(property "Reference" "#PWR084"
 			(at 58.42 118.11 0)
 			(hide yes)
@@
 			(project "motor_testbench_v1_0"
 				(path "/da638649-102c-44f9-b928-e91cd399cc2f/f4ebbd2c-ae23-469d-a040-5f643f36c41b"
-					(reference "#PWR083")
+					(reference "#PWR084")
 					(unit 1)
 				)
@@
 		(in_pos_files yes)
 		(dnp no)
-		(property "Reference" "#PWR085"
+		(property "Reference" "#PWR086"
 			(at 60.96 172.72 0)
 			(hide yes)
@@
 			(project "motor_testbench_v1_0"
 				(path "/da638649-102c-44f9-b928-e91cd399cc2f/f4ebbd2c-ae23-469d-a040-5f643f36c41b"
-					(reference "#PWR085")
+					(reference "#PWR086")
 					(unit 1)
 				)
@@
 	(symbol
 		(lib_id "Device:C")
-		(at 449.58 166.37 180)
+		(at 365.76 -24.13 180)
 		(unit 1)
 		(body_style 1)
@@
 		(dnp no)
 		(property "Reference" "C113"
-			(at 447.04 164.084 0)
+			(at 363.22 -26.416 0)
 			(show_name no)
 			(do_not_autoplace no)
@@
 		)
 		(property "Value" "1u"
-			(at 447.04 161.798 0)
+			(at 363.22 -28.702 0)
 			(show_name no)
 			(do_not_autoplace no)
@@
 		)
 		(property "Footprint" "Capacitor_SMD:C_0603_1608Metric_Pad1.08x0.95mm_HandSolder"
-			(at 448.6148 162.56 0)
+			(at 364.7948 -27.94 0)
 			(hide yes)
 			(show_name no)
@@
 		)
 		(property "Datasheet" ""
-			(at 449.58 166.37 0)
+			(at 365.76 -24.13 0)
 			(hide yes)
 			(show_name no)
@@
 		)
 		(property "Description" "Unpolarized capacitor"
-			(at 449.58 166.37 0)
+			(at 365.76 -24.13 0)
 			(hide yes)
 			(show_name no)
@@
 		)
 		(property "Manufacturing_Number" ""
-			(at 449.58 166.37 0)
+			(at 365.76 -24.13 0)
 			(hide yes)
 			(show_name no)
@@
 		(dnp no)
 		(fields_autoplaced yes)
-		(property "Reference" "#PWR084"
+		(property "Reference" "#PWR085"
 			(at 60.96 139.7 0)
 			(hide yes)
@@
 			(project "motor_testbench_v1_0"
 				(path "/da638649-102c-44f9-b928-e91cd399cc2f/f4ebbd2c-ae23-469d-a040-5f643f36c41b"
-					(reference "#PWR084")
+					(reference "#PWR085")
 					(unit 1)
 				)
@@
 	(symbol
 		(lib_id "Device:R")
-		(at 449.58 149.86 0)
+		(at 365.76 -40.64 0)
 		(unit 1)
 		(body_style 1)
@@
 		(dnp no)
 		(property "Reference" "R45"
-			(at 436.372 147.8281 0)
+			(at 352.552 -42.6719 0)
 			(show_name no)
 			(do_not_autoplace no)
@@
 		)
 		(property "Value" "10k"
-			(at 436.372 150.3681 0)
+			(at 352.552 -40.1319 0)
 			(show_name no)
 			(do_not_autoplace no)
@@
 		)
 		(property "Footprint" "Resistor_SMD:R_0603_1608Metric_Pad0.98x0.95mm_HandSolder"
-			(at 447.802 149.86 90)
+			(at 363.982 -40.64 90)
 			(hide yes)
 			(show_name no)
@@
 		)
 		(property "Datasheet" ""
-			(at 449.58 149.86 0)
+			(at 365.76 -40.64 0)
 			(hide yes)
 			(show_name no)
@@
 		)
 		(property "Description" "Resistor"
-			(at 449.58 149.86 0)
+			(at 365.76 -40.64 0)
 			(hide yes)
 			(show_name no)
@@
 		)
 		(property "Manufacturing_Number" ""
-			(at 449.58 149.86 0)
+			(at 365.76 -40.64 0)
 			(hide yes)
 			(show_name no)

Commit message: Continue implementing ESP32 module
[KiCad Version: 10.0.3]
Parts:
- removed C72: 1u, Capacitor_SMD:C_0603_1608Metric_Pad1.08x0.95mm_HandSolder, symbol Device:C
- removed U12: TLV75733PDYDR, Package_TO_SOT_SMD:SOT-23-5, symbol Regulator_Linear:TLV75733PDBV
- added U14: TLV75733PDYDR, Package_TO_SOT_SMD:SOT-23-5, symbol Regulator_Linear:TLV75733PDBV
- added U2: AP7361C-33Y5-13, Package_TO_SOT_SMD:SOT-89-5_Handsoldering, symbol Regulator_Linear:AP7361C-33E
- C69: value 1u -> 10u
- renumbered C113 to C109, C109 to C110, C110 to C111, C111 to C112, C112 to C113, D5 to D6, D6 to D7, D7 to D8, D8 to D9, R24 to R25, R25 to R26, R26 to R27, R27 to R28, R28 to R29, R29 to R30, R30 to R31, R31 to R32, R32 to R33, R33 to R34, R34 to R35, R35 to R36, R36 to R37, R37 to R38, R38 to R39, R39 to R40, R40 to R41, R41 to R42, R42 to R43, R43 to R44, R44 to R45, R45 to R46, U8 to U10, U9 to U11, U10 to U12, U11 to U13, U13 to U15, U14 to U16, U15 to U17, U16 to U18, U17 to U19, U18 to U20, U19 to U21, U7 to U9
Connections:
- net +3V3_ESP: now also U2.5 (VOUT)
- net +6V_Buck_Out: now also U2.4 (VIN)
- net GND: now also U2.2 (GND)
- net at C73.2, R36.2: now also U2.1 (EN)
- no-connect marks 0 -> 1
Other:
- moved on the sheet: C53, C78

Commit message: Add new GPIO header. Minor improvements.
[KiCad Version: 10.0.3]
Parts:
- removed C95: 1u, Capacitor_SMD:C_0603_1608Metric_Pad1.08x0.95mm_HandSolder, symbol Device:C
- removed DIO1: TestPoint, TestPoint:TestPoint_Pad_D1.0mm, symbol Connector:TestPoint
- removed J12: Conn_01x02_Pin, Connector_PinHeader_2.54mm:PinHeader_1x02_P2.54mm_Vertical, symbol Connector:Conn_01x02_Pin

Commit message: Add buffer OPA for Secondary battery measurement
[KiCad Version: 10.0.3]
Parts:
- removed D7: SK15, Diode_SMD:D_SMA, symbol Device:D_Schottky
- added C133: 10u, Capacitor_SMD:C_0603_1608Metric_Pad1.08x0.95mm_HandSolder, symbol Device:C
- added C66: 1u, Capacitor_SMD:C_0603_1608Metric_Pad1.08x0.95mm_HandSolder, symbol Device:C
- added D10, D9: SB56AFC-AU_R1_000A1, Diode_SMD:D_SMA, symbol Device:D_Schottky
- added J9: Conn_01x02_Pin, Connector_PinHeader_2.54mm:PinHeader_1x02_P2.54mm_Vertical, symbol Connector:Conn_01x02_Pin
- renumbered C96 to C100, C97 to C101, C98 to C102, C99 to C103, C100 to C104, C101 to C105, C102 to C106, C103 to C107, C104 to C108, C105 to C109, C106 to C110, C107 to C111, C108 to C112, C109 to C113, C110 to C114, C111 to C115, C112 to C116, C113 to C117, C45 to C50, C46 to C51, C47 to C52, C48 to C53, C49 to C54, C50 to C55, C51 to C56, C52 to C57, C53 to C58, C54 to C59, C55 to C60, C56 to C61, C57 to C62, C58 to C63, C59 to C64, C60 to C65, C61 to C67, C62 to C68, C63 to C69, C64 to C70, C65 to C71, C66 to C72, C67 to C73, C68 to C74, C69 to C75, C70 to C76, C71 to C77, C73 to C78, C74 to C79, C75 to C80, C76 to C81, C77 to C82, C78 to C83, C79 to C84, C80 to C85, C81 to C86, C82 to C87, C83 to C88, C84 to C89, C85 to C90, C86 to C91, C87 to C92, C88 to C93, C89 to C94, C90 to C95, C91 to C96, C92 to C97, C93 to C98, C94 to C99, D8 to D11, D9 to D12, D6 to D8, DIO2 to DIO1, J13 to J10, J10 to J7, J11 to J8, R25 to R39, R26 to R40, R27 to R41, R28 to R42, R29 to R43, R30 to R44, R31 to R45, R32 to R46, R33 to R47, R34 to R48, R35 to R49, R36 to R50, R37 to R51, R38 to R52, R39 to R53, R40 to R54, R41 to R55, R42 to R56, R43 to R57, R44 to R58, R45 to R59, R46 to R60, U12 to U10, U13 to U11, U2 to U12, U15 to U13, U16 to U14, U17 to U15, U14 to U16, U18 to U17, U19 to U18, U20 to U19, U21 to U20, U9 to U7, U10 to U8, U11 to U9
Connections:
- net +12V_Fan_Supply: now also D10.2 (A)
- net +3V3_ESP: now also C133.2
- net +6V_Buck_Out: now also C66.2, J9.1 (Pin_1)
- net +VBat_Secondary: now also D9.1 (K); no longer D8.1 (K), D8.2 (K), J7.2 (Pin_2)
- net GND: now also C133.1, C66.1, J9.2 (Pin_2)
- net at C63.2, J8.1 (Pin_1), L1.2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: now also D10.1 (K)
- new net: D8.1 (K), D8.2 (K), D9.2 (A), J7.2 (Pin_2)
